File: MainPlatine/motor.kicad_sch (KiCad schematic)
At the start: 1 part

Commit message: add new
Parts:
- Motor1: footprint Connector_PinSocket_2.54mm:PinSocket_1x06_P2.54mm_Vertical -> JST:JST-XH-06-PACKAGE-LONG-PAD
Changed lines of the file:
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@@
 		(instances
 			(project "MainPlatine"
-				(path "/68a83b6d-2c86-4b88-bf4a-0c6f931ae55b/e73857bf-05f8-4db1-9dd6-dfa24c8b2cae/0df11882-2d85-4dca-ba7b-f69dbb9d7361"
-					(reference "#PWR025")
+				(path "/68a83b6d-2c86-4b88-bf4a-0c6f931ae55b/cc08bab7-5b58-4988-96a3-a32e29019015/05ba44bc-ea1f-4207-adbb-a2ff860ae7b9"
+					(reference "#PWR023")
 					(unit 1)
 				)
-				(path "/68a83b6d-2c86-4b88-bf4a-0c6f931ae55b/e73857bf-05f8-4db1-9dd6-dfa24c8b2cae/470ae657-6e50-4fa8-9b97-34138efdb176"
+				(path "/68a83b6d-2c86-4b88-bf4a-0c6f931ae55b/cc08bab7-5b58-4988-96a3-a32e29019015/d8bad468-1a27-44c2-8297-3d2f1968dea5"
+					(reference "#PWR022")
+					(unit 1)
+				)
+				(path "/68a83b6d-2c86-4b88-bf4a-0c6f931ae55b/d531c041-0bbf-46c1-9e17-ec91239c9bac/05ba44bc-ea1f-4207-adbb-a2ff860ae7b9"
 					(reference "#PWR027")
 					(unit 1)
 				)
-				(path "/68a83b6d-2c86-4b88-bf4a-0c6f931ae55b/fdc0243a-a5a5-4468-9cc0-28e8593b5b3d/0df11882-2d85-4dca-ba7b-f69dbb9d7361"
-					(reference "#PWR022")
-					(unit 1)
-				)
-				(path "/68a83b6d-2c86-4b88-bf4a-0c6f931ae55b/fdc0243a-a5a5-4468-9cc0-28e8593b5b3d/470ae657-6e50-4fa8-9b97-34138efdb176"
-					(reference "#PWR023")
+				(path "/68a83b6d-2c86-4b88-bf4a-0c6f931ae55b/d531c041-0bbf-46c1-9e17-ec91239c9bac/d8bad468-1a27-44c2-8297-3d2f1968dea5"
+					(reference "#PWR025")
 					(unit 1)
 				)
@@
 		(instances
 			(project "MainPlatine"
-				(path "/68a83b6d-2c86-4b88-bf4a-0c6f931ae55b/e73857bf-05f8-4db1-9dd6-dfa24c8b2cae/0df11882-2d85-4dca-ba7b-f69dbb9d7361"
-					(reference "#PWR024")
+				(path "/68a83b6d-2c86-4b88-bf4a-0c6f931ae55b/cc08bab7-5b58-4988-96a3-a32e29019015/05ba44bc-ea1f-4207-adbb-a2ff860ae7b9"
+					(reference "#PWR021")
 					(unit 1)
 				)
-				(path "/68a83b6d-2c86-4b88-bf4a-0c6f931ae55b/e73857bf-05f8-4db1-9dd6-dfa24c8b2cae/470ae657-6e50-4fa8-9b97-34138efdb176"
+				(path "/68a83b6d-2c86-4b88-bf4a-0c6f931ae55b/cc08bab7-5b58-4988-96a3-a32e29019015/d8bad468-1a27-44c2-8297-3d2f1968dea5"
+					(reference "#PWR020")
+					(unit 1)
+				)
+				(path "/68a83b6d-2c86-4b88-bf4a-0c6f931ae55b/d531c041-0bbf-46c1-9e17-ec91239c9bac/05ba44bc-ea1f-4207-adbb-a2ff860ae7b9"
 					(reference "#PWR026")
 					(unit 1)
 				)
-				(path "/68a83b6d-2c86-4b88-bf4a-0c6f931ae55b/fdc0243a-a5a5-4468-9cc0-28e8593b5b3d/0df11882-2d85-4dca-ba7b-f69dbb9d7361"
-					(reference "#PWR020")
-					(unit 1)
-				)
-				(path "/68a83b6d-2c86-4b88-bf4a-0c6f931ae55b/fdc0243a-a5a5-4468-9cc0-28e8593b5b3d/470ae657-6e50-4fa8-9b97-34138efdb176"
-					(reference "#PWR021")
+				(path "/68a83b6d-2c86-4b88-bf4a-0c6f931ae55b/d531c041-0bbf-46c1-9e17-ec91239c9bac/d8bad468-1a27-44c2-8297-3d2f1968dea5"
+					(reference "#PWR024")
 					(unit 1)
 				)
@@
 			)
 		)
-		(property "Footprint" "Connector_PinSocket_2.54mm:PinSocket_1x06_P2.54mm_Vertical"
+		(property "Footprint" "JST:JST-XH-06-PACKAGE-LONG-PAD"
 			(at 139.7 104.14 0)
 			(effects
@@
 		(instances
 			(project "MainPlatine"
-				(path "/68a83b6d-2c86-4b88-bf4a-0c6f931ae55b/e73857bf-05f8-4db1-9dd6-dfa24c8b2cae/0df11882-2d85-4dca-ba7b-f69dbb9d7361"
+				(path "/68a83b6d-2c86-4b88-bf4a-0c6f931ae55b/cc08bab7-5b58-4988-96a3-a32e29019015/05ba44bc-ea1f-4207-adbb-a2ff860ae7b9"
+					(reference "Motor2")
+					(unit 1)
+				)
+				(path "/68a83b6d-2c86-4b88-bf4a-0c6f931ae55b/cc08bab7-5b58-4988-96a3-a32e29019015/d8bad468-1a27-44c2-8297-3d2f1968dea5"
+					(reference "Motor1")
+					(unit 1)
+				)
+				(path "/68a83b6d-2c86-4b88-bf4a-0c6f931ae55b/d531c041-0bbf-46c1-9e17-ec91239c9bac/05ba44bc-ea1f-4207-adbb-a2ff860ae7b9"
+					(reference "Motor4")
+					(unit 1)
+				)
+				(path "/68a83b6d-2c86-4b88-bf4a-0c6f931ae55b/d531c041-0bbf-46c1-9e17-ec91239c9bac/d8bad468-1a27-44c2-8297-3d2f1968dea5"
 					(reference "Motor3")
 					(unit 1)
 				)
-				(path "/68a83b6d-2c86-4b88-bf4a-0c6f931ae55b/e73857bf-05f8-4db1-9dd6-dfa24c8b2cae/470ae657-6e50-4fa8-9b97-34138efdb176"
-					(reference "Motor4")
-					(unit 1)
-				)
-				(path "/68a83b6d-2c86-4b88-bf4a-0c6f931ae55b/fdc0243a-a5a5-4468-9cc0-28e8593b5b3d/0df11882-2d85-4dca-ba7b-f69dbb9d7361"
-					(reference "Motor1")
-					(unit 1)
-				)
-				(path "/68a83b6d-2c86-4b88-bf4a-0c6f931ae55b/fdc0243a-a5a5-4468-9cc0-28e8593b5b3d/470ae657-6e50-4fa8-9b97-34138efdb176"
-					(reference "Motor2")
-					(unit 1)
-				)
