File: MainPlatine/treiber.kicad_sch (KiCad schematic)
At the start: 1 part, among them U4 TB6612FNG

Commit message: add new
Connections:
- net B+: now also U4.7 (BO2), U4.8 (BO2); no longer U4.11 (BO1), U4.12 (BO1)
- net B-: now also U4.11 (BO1), U4.12 (BO1); no longer U4.7 (BO2), U4.8 (BO2)
Changed lines of the file:
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@@
+	(wire
+		(pts
+			(xy 168.91 81.28) (xy 176.53 81.28)
+		)
+		(stroke
+			(width 0)
+			(type default)
+		)
+	)
+	(wire
+		(pts
+			(xy 124.46 119.38) (xy 124.46 121.92)
+		)
+		(stroke
+			(width 0)
+			(type default)
+		)
+	)
+	(wire
+		(pts
+			(xy 129.54 60.96) (xy 129.54 64.77)
+		)
+		(stroke
+			(width 0)
+			(type default)
+		)
+	)
 	(wire
 		(pts
@@
 	(wire
 		(pts
-			(xy 168.91 81.28) (xy 176.53 81.28)
-		)
-		(stroke
-			(width 0)
-			(type default)
-		)
-	)
-	(wire
-		(pts
-			(xy 124.46 119.38) (xy 124.46 121.92)
-		)
-		(stroke
-			(width 0)
-			(type default)
-		)
-	)
-	(wire
-		(pts
-			(xy 129.54 60.96) (xy 129.54 64.77)
-		)
-		(stroke
-			(width 0)
-			(type default)
-		)
-	)
-	(wire
-		(pts
 			(xy 102.87 82.55) (xy 109.22 82.55)
 		)
@@
 	(wire
 		(pts
+			(xy 139.7 95.25) (xy 144.78 95.25)
+		)
+		(stroke
+			(width 0)
+			(type default)
+		)
+	)
+	(wire
+		(pts
 			(xy 132.08 119.38) (xy 127 119.38)
 		)
@@
 			(width 0)
 			(type default)
-		)
-	)
-	(wire
-		(pts
-			(xy 139.7 95.25) (xy 144.78 95.25)
-		)
-		(stroke
-			(width 0)
-			(type default)
-		)
-	)
-	(label "B+"
-		(at 144.78 95.25 180)
-		(effects
-			(font
-				(size 1.27 1.27)
-			)
-			(justify right bottom)
-		)
-	)
-	(label "B-"
-		(at 144.78 100.33 180)
-		(effects
-			(font
-				(size 1.27 1.27)
-			)
-			(justify right bottom)
 		)
 	)
@@
 		)
 	)
+	(label "B+"
+		(at 144.78 100.33 180)
+		(effects
+			(font
+				(size 1.27 1.27)
+			)
+			(justify right bottom)
+		)
+	)
 	(label "A+"
 		(at 144.78 82.55 180)
@@
 			)
 			(justify left bottom)
+		)
+	)
+	(label "B-"
+		(at 144.78 95.25 180)
+		(effects
+			(font
+				(size 1.27 1.27)
+			)
+			(justify right bottom)
 		)
 	)
@@
 		(instances
 			(project "MainPlatine"
-				(path "/68a83b6d-2c86-4b88-bf4a-0c6f931ae55b/e73857bf-05f8-4db1-9dd6-dfa24c8b2cae"
+				(path "/68a83b6d-2c86-4b88-bf4a-0c6f931ae55b/cc08bab7-5b58-4988-96a3-a32e29019015"
+					(reference "#PWR04")
+					(unit 1)
+				)
+				(path "/68a83b6d-2c86-4b88-bf4a-0c6f931ae55b/d531c041-0bbf-46c1-9e17-ec91239c9bac"
 					(reference "#PWR05")
-					(unit 1)
-				)
-				(path "/68a83b6d-2c86-4b88-bf4a-0c6f931ae55b/fdc0243a-a5a5-4468-9cc0-28e8593b5b3d"
-					(reference "#PWR04")
 					(unit 1)
 				)
@@
 		(instances
 			(project "MainPlatine"
-				(path "/68a83b6d-2c86-4b88-bf4a-0c6f931ae55b/e73857bf-05f8-4db1-9dd6-dfa24c8b2cae"
+				(path "/68a83b6d-2c86-4b88-bf4a-0c6f931ae55b/cc08bab7-5b58-4988-96a3-a32e29019015"
+					(reference "U4")
+					(unit 1)
+				)
+				(path "/68a83b6d-2c86-4b88-bf4a-0c6f931ae55b/d531c041-0bbf-46c1-9e17-ec91239c9bac"
 					(reference "U5")
-					(unit 1)
-				)
-				(path "/68a83b6d-2c86-4b88-bf4a-0c6f931ae55b/fdc0243a-a5a5-4468-9cc0-28e8593b5b3d"
-					(reference "U4")
 					(unit 1)
 				)
@@
 		(instances
 			(project "MainPlatine"
-				(path "/68a83b6d-2c86-4b88-bf4a-0c6f931ae55b/e73857bf-05f8-4db1-9dd6-dfa24c8b2cae"
+				(path "/68a83b6d-2c86-4b88-bf4a-0c6f931ae55b/cc08bab7-5b58-4988-96a3-a32e29019015"
+					(reference "#PWR06")
+					(unit 1)
+				)
+				(path "/68a83b6d-2c86-4b88-bf4a-0c6f931ae55b/d531c041-0bbf-46c1-9e17-ec91239c9bac"
 					(reference "#PWR07")
-					(unit 1)
-				)
-				(path "/68a83b6d-2c86-4b88-bf4a-0c6f931ae55b/fdc0243a-a5a5-4468-9cc0-28e8593b5b3d"
-					(reference "#PWR06")
 					(unit 1)
 				)
@@
 			(color 0 0 0 0.0000)
 		)
-		(property "Sheetname" "Motor1"
+		(property "Sheetname" "Motor2"
 			(at 176.53 71.6784 0)
 			(effects
@@
 		(instances
 			(project "MainPlatine"
-				(path "/68a83b6d-2c86-4b88-bf4a-0c6f931ae55b/fdc0243a-a5a5-4468-9cc0-28e8593b5b3d"
-					(page "5")
-				)
-				(path "/68a83b6d-2c86-4b88-bf4a-0c6f931ae55b/e73857bf-05f8-4db1-9dd6-dfa24c8b2cae"
-					(page "7")
+				(path "/68a83b6d-2c86-4b88-bf4a-0c6f931ae55b/cc08bab7-5b58-4988-96a3-a32e29019015"
+					(page "6")
+				)
+				(path "/68a83b6d-2c86-4b88-bf4a-0c6f931ae55b/d531c041-0bbf-46c1-9e17-ec91239c9bac"
+					(page "8")
 				)
 			)
@@
 			(color 0 0 0 0.0000)
 		)
-		(property "Sheetname" "Motor2"
+		(property "Sheetname" "Motor1"
 			(at 176.53 93.2684 0)
 			(effects
@@
 		(instances
 			(project "MainPlatine"
-				(path "/68a83b6d-2c86-4b88-bf4a-0c6f931ae55b/fdc0243a-a5a5-4468-9cc0-28e8593b5b3d"
-					(page "6")
-				)
-				(path "/68a83b6d-2c86-4b88-bf4a-0c6f931ae55b/e73857bf-05f8-4db1-9dd6-dfa24c8b2cae"
-					(page "8")
-				)
-			)
+				(path "/68a83b6d-2c86-4b88-bf4a-0c6f931ae55b/cc08bab7-5b58-4988-96a3-a32e29019015"
+					(page "5")
+				)
+				(path "/68a83b6d-2c86-4b88-bf4a-0c6f931ae55b/d531c041-0bbf-46c1-9e17-ec91239c9bac"
+					(page "7")
+				)
+			)
