File: MainPlatine/MainPlatine.kicad_sch (KiCad schematic)
At the start: 1 part

Commit message: add new
Parts:
- added RI1, RI2: 10k, Resistor_SMD:R_1206_3216Metric_Pad1.30x1.75mm_HandSolder, symbol Device:R
- added U1: Main Conector to Main pcb, Robotik:Main Conetor, symbol RobotikV4:MainConector
Connections:
- net +5V: now also RI1.1, RI2.1, U1.5V
- net GND: now also U1.GND
- net MOT1_IN1: now also B1.31; no longer B1.25
- net MOT1_IN2: now also B1.29; no longer B1.27
- net MOT2_IN1: now also B1.23; no longer B1.29
- net MOT2_IN2: now also B1.25; no longer B1.31
- net MOT3_IN1: now also B1.49; no longer B1.33
- net MOT3_IN2: now also B1.47; no longer B1.35
- net MOT4_IN1: now also B1.43; no longer B1.37
- net MOT4_IN2: now also B1.45; no longer B1.39
- net MOT_STBY: now also B1.27; no longer B1.23
- net ARD_RX_3: now reaches B1.14 (14(TX3))
- net ARD_TX_3: now reaches B1.15 (15(RX3))
- net ARD_TX_2: now reaches B1.16 (16(TX2))
- net ARD_TX_2: now also U1.RX_C2 (RX_Cam_2)
- net ARD_RX_2: now reaches B1.17 (17(RX2))
- net ARD_RX_2: now also U1.TX_C2 (TX_Cam_2)
- net ARD_TX_1: now reaches B1.18 (18(TX1))
- net ARD_TX_1: now also U1.RX_C1 (RX_Cam_1)
- net ARD_RX_1: now reaches B1.19 (19(RX1))
- net ARD_RX_1: now also U1.TX_C1 (TX_Cam_1)
- net Bumper_Links: now reaches B1.2
- net SDA: now reaches B1.20 (20(SDA))
- net SDA: now also RI1.2, U1.SDA
- net SCL: now reaches B1.21 (21(SCL))
- net SCL: now also RI2.2, U1.SCL
- net Bumper_Rechts: now reaches B1.3
- net Tof_XS_0: now reaches B1.30
- net Tof_XS_4: now reaches B1.32
- net Tof_XS_4: now also U1.TXS1 (ToF_XS_1)
- net Tof_XS_5: now reaches B1.34
- net Tof_XS_5: now also U1.TXS2 (ToF_XS_2)
- net Tof_XS_6: now reaches B1.36
- net Tof_XS_6: now also U1.TXS3 (ToF_XS_3)
- net LED_C2: now reaches B1.38
- net LED_C2: now also U1.LED1 (Beleuchtung_Cam_1)
- net LED_C1: now reaches B1.40
- net LED_C1: now also U1.LED2 (Beleuchtung_Cam_2)
- net Tof_XS_3: now reaches B1.41
- net UI_LED_2: now reaches B1.42
- net UI_LED_2: now also U1.LED_B (UI_Led_2)
- net UI_LED_1: now reaches B1.44
- net UI_LED_1: now also U1.LED_A (UI_Led_1)
- net UI_Button_3: now reaches B1.A0
- net UI_Button_3: now also U1.UI_B3 (UI_Button_3)
- net UI_Button_4: now reaches B1.A1
- net UI_Button_4: now also U1.UI_B4 (UI_Button_4)
- net Encoder_B: now reaches B1.A10
- net Encoder_B: now also U1.RE_B (Encoder_B)
- net Encoder_SW: now reaches B1.A11
- net Encoder_SW: now also U1.RE_SW (Encoder_Taster)
- net Encoder_A: now reaches B1.A12
- net Encoder_A: now also U1.RE_A (Encoder_A)
- net UI_Button_2: now reaches B1.A13
- net UI_Button_2: now also U1.UI_B2 (UI_Button_2)
- net UI_Button_1: now reaches B1.A14
- net UI_Button_1: now also U1.UI_B1 (UI_Button_1)
- net Color_Old_Interrupt: now reaches B1.A15
- net Interrupt_Cam1: now reaches B1.A8
- net Interrupt_Cam1: now also U1.I_C2 (Interrupt_Cam_2)
- net Interrupt_Cam2: now reaches B1.A9
- net Interrupt_Cam2: now also U1.I_C1 (Interrupt_Cam_1)
- new net SW_SCL: B1.33
- new net SW_SDA: B1.35
- new net Tof_XS_1: B1.37
- new net Tof_XS_2: B1.39
- no-connect marks 0 -> 8
Other:
- added sheet Encoder_Unit (encoder.kicad_sch)
- sheet Sensorik ports: added Bumper_Links, Bumper_Rechts, Color_Old_Int; removed Bumper_1, Bumper_2, Color_Old_IO, ToF_XS_4, ToF_XS_5, ToF_XS_6

Commit message: add main PCB
Parts:
- added J2: Conn_01x02_Pin, JST:JST-XH-02-PACKAGE-LONG-PAD, symbol Connector:Conn_01x02_Pin
- added J3: Conn_01x04_Pin, symbol Connector:Conn_01x04_Pin
Connections:
- net +5V: now also J3.1 (Pin_1)
- net Akku: now also J2.1 (Pin_1)
- net GND: now also J2.2 (Pin_2), J3.4 (Pin_4)
- net LEDB_U: now reaches B1.26
- net GYRO_RST: now reaches B1.28
- net MISO: now reaches B1.50 (50/MISO)
- net MISO: now also U1.MOSI
- net MOSI: now reaches B1.51 (51/MOSI)
- net MOSI: now also U1.MISO
- net SCK: now reaches B1.52 (52/SCK)
- net SCK: now also U1.SCK
- net D+: now reaches U1.D+ (Mega_D+)
- net D+: now also J3.2 (Pin_2)
- net D-: now reaches U1.D- (Mega_D-)
- net D-: now also J3.3 (Pin_3)
Other:
- sheet PowerSupplyUnit ports: added none; removed AKKU_ENA

Commit message: fix main pcb
Connections:
- net BAT_ADC: now also B1.A7
- net Color_NEW_IO: now also B1.48
- net GYRO_RST: now also B1.24; no longer B1.28
- net LEDB_U: now also B1.22; no longer B1.26
- net D_D: now reaches B1.46
- net D_D: now also U1.D_D (D_Display)
- net CS_D: now reaches B1.53 (53/~{CS})
- net CS_D: now also U1.CS_D (CS_Display)
- net IO_CAM1: now reaches U1.R_C1 (Reset_Cam_1)
- net IO_CAM1: now also B1.28
- net IO_CAM2: now reaches U1.R_C2 (Reset_Cam_2)
- net IO_CAM2: now also B1.26
- no-connect marks 8 -> 15

Commit message: update new
Parts:
- added RS_1, RS_2: Conn_01x03_Pin, JST:JST-XH-03-PACKAGE-LONG-PAD, symbol Connector:Conn_01x03_Pin
Connections:
- net +5V: now also RS_1.1 (Pin_1), RS_2.1 (Pin_1)
- net ARD_RX_1: no longer U1.TX_C1 (TX_Cam_1)
- net ARD_TX_1: no longer U1.RX_C1 (RX_Cam_1)
- net GND: now also RS_1.3 (Pin_3), RS_2.3 (Pin_3)
- net IO_CAM1: no longer U1.R_C1 (Reset_Cam_1)
- net Interrupt_Cam2: no longer U1.I_C1 (Interrupt_Cam_1)
- net LED_C2: no longer U1.LED1 (Beleuchtung_Cam_1)
- net RS_Servo_1: now reaches B1.10
- net RS_Servo_1: now also RS_1.2 (Pin_2)
- net RES_D: now reaches B1.8
- net RES_D: now also U1.1 (RES_D)
- net RS_Servo_2: now reaches B1.9
- net RS_Servo_2: now also RS_2.2 (Pin_2)
