File: MainPlatine/sensorik.kicad_sch (KiCad schematic)
At the start: 13 parts

Commit message: add new
Parts:
- removed ToF_Bus_H2, ToF_Bus_V1: Conn_01x04_Pin, symbol Connector:Conn_01x04_Pin
- removed ToF_Vorne_U1: Conn_01x05_Pin, symbol Connector:Conn_01x05_Pin
- removed Tof_XS_H1, Tof_XS_V1: Conn_01x03_Pin, symbol Connector:Conn_01x03_Pin
- added J1: Conn_01x07_Pin, JST:JST-XH-07-PACKAGE-LONG-PAD, symbol Connector:Conn_01x07_Pin
- added ToF_Vorne_1: Conn_01x06_Socket, Connector_PinSocket_2.54mm:PinSocket_1x06_P2.54mm_Horizontal, symbol Connector:Conn_01x06_Socket
- Bumper_1, Bumper_2: footprint (none) -> JST:JST-XH-02-PACKAGE-LONG-PAD
- Colo_Alt1: renamed from Colo_Alt; footprint (none) -> JST:JST-XH-05-PACKAGE-LONG-PAD
- Color_NEU1: renamed from Color_NEU; footprint (none) -> JST:JST-XH-05-PACKAGE-LONG-PAD
- Gyro1: renamed from Gyro; footprint (none) -> JST:JST-XH-05-PACKAGE-LONG-PAD
- LED_Color1: renamed from LED_Color; footprint (none) -> JST:JST-XH-03PACKAGE-LONG-PAD
Connections:
- net +5V: now also J1.6 (Pin_6), ToF_Vorne_1.6 (Pin_6)
- net GND: now also J1.7 (Pin_7), ToF_Vorne_1.5 (Pin_5)
- net SCL: now also J1.5 (Pin_5), ToF_Vorne_1.4 (Pin_4)
- net SDA: now also J1.4 (Pin_4), ToF_Vorne_1.3 (Pin_3)
- net ToF_XS_0: now also ToF_Vorne_1.1 (Pin_1)
- net ToF_XS_1: now also J1.1 (Pin_1)
- net ToF_XS_2: now also J1.2 (Pin_2)
- net ToF_XS_3: now also J1.3 (Pin_3)
- net Bumper_1 renamed Bumper_Links
- net Bumper_2 renamed Bumper_Rechts
- net Color_Old_IO renamed Color_Old_Int
- no-connect marks 0 -> 1

Commit message: add main PCB
Parts:
- removed LED_Color1: Conn_01x03_Pin, JST:JST-XH-03PACKAGE-LONG-PAD, symbol Connector:Conn_01x03_Pin
- added J4: Conn_01x03_Pin, JST:JST-XH-03-PACKAGE-LONG-PAD, symbol Connector:Conn_01x03_Pin
Connections:
- net +5V: now also J1.2 (Pin_2), J4.1 (Pin_1); no longer J1.6 (Pin_6)
- net GND: now also J1.1 (Pin_1), J4.3 (Pin_3); no longer J1.7 (Pin_7)
- net LED_Beleuchtung_Unten: now also J4.2 (Pin_2)
- net SCL: now also J1.3 (Pin_3); no longer J1.5 (Pin_5)
- net ToF_XS_1: now also J1.7 (Pin_7); no longer J1.1 (Pin_1)
- net ToF_XS_2: now also J1.6 (Pin_6); no longer J1.2 (Pin_2)
- net ToF_XS_3: now also J1.5 (Pin_5); no longer J1.3 (Pin_3)
Changed lines of the file:
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@@
 		(lib_id "Connector:Conn_01x07_Pin")
 		(at 151.13 67.31 0)
-		(unit 1)
-		(exclude_from_sim no)
-		(in_bom yes)
-		(on_board yes)
-		(dnp no)
-		(fields_autoplaced yes)
+		(mirror x)
+		(unit 1)
+		(exclude_from_sim no)
+		(in_bom yes)
+		(on_board yes)
+		(dnp no)
 		(property "Reference" "J1"
-			(at 151.765 54.61 0)
-			(effects
-				(font
-					(size 1.27 1.27)
-				)
+			(at 149.86 66.0399 0)
+			(effects
+				(font
+					(size 1.27 1.27)
+				)
+				(justify right)
 			)
 		)
 		(property "Value" "Conn_01x07_Pin"
-			(at 151.765 57.15 0)
-			(effects
-				(font
-					(size 1.27 1.27)
-				)
+			(at 149.86 68.5799 0)
+			(effects
+				(font
+					(size 1.27 1.27)
+				)
+				(justify right)
 			)
 		)
@@
 		)
 		(instances
-			(project ""
+			(project "MainPlatine"
 				(path "/68a83b6d-2c86-4b88-bf4a-0c6f931ae55b/b5cdc453-d330-4215-a4bc-cc85e155168a"
 					(reference "J1")
@@
 		(on_board yes)
 		(dnp no)
-		(property "Reference" "LED_Color1"
-			(at 197.866 106.68 90)
+		(fields_autoplaced yes)
+		(property "Reference" "J4"
+			(at 200.025 99.06 0)
 			(effects
 				(font
@@
 					(size 1.27 1.27)
 				)
-				(hide yes)
-			)
-		)
-		(property "Footprint" "JST:JST-XH-03PACKAGE-LONG-PAD"
+			)
+		)
+		(property "Footprint" "JST:JST-XH-03-PACKAGE-LONG-PAD"
 			(at 199.39 106.68 0)
 			(effects
@@
 		(pin "3"
 		)
+		(pin "1"
+		)
 		(pin "2"
 		)
-		(pin "1"
-		)
-		(instances
-			(project "MainPlatine"
-				(path "/68a83b6d-2c86-4b88-bf4a-0c6f931ae55b/b5cdc453-d330-4215-a4bc-cc85e155168a"
-					(reference "LED_Color1")
-					(unit 1)
-				)
+		(instances
+			(project ""
+				(path "/68a83b6d-2c86-4b88-bf4a-0c6f931ae55b/b5cdc453-d330-4215-a4bc-cc85e155168a"
+					(reference "J4")
+					(unit 1)
+				)

Commit message: fix main pcb
Connections:
- net +5V: now also ToF_Vorne_1.1 (Pin_1); no longer ToF_Vorne_1.6 (Pin_6)
- net GND: now also ToF_Vorne_1.2 (Pin_2); no longer ToF_Vorne_1.5 (Pin_5)
- net SCL: now also ToF_Vorne_1.3 (Pin_3); no longer ToF_Vorne_1.4 (Pin_4)
- net SDA: now also ToF_Vorne_1.4 (Pin_4); no longer ToF_Vorne_1.3 (Pin_3)
- net ToF_XS_0: now also ToF_Vorne_1.6 (Pin_6); no longer ToF_Vorne_1.1 (Pin_1)
Other:
- moved on the sheet: ToF_Vorne_1
Changed lines of the file:
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@@
 	(symbol
 		(lib_id "Connector:Conn_01x06_Socket")
-		(at 68.58 69.85 180)
+		(at 68.58 67.31 0)
+		(mirror y)
 		(unit 1)
 		(exclude_from_sim no)
@@
 		)
 		(property "Value" "Conn_01x06_Socket"
-			(at 69.215 59.69 0)
+			(at 69.215 77.47 0)
 			(effects
 				(font
@@
 		)
 		(property "Footprint" "Connector_PinSocket_2.54mm:PinSocket_1x06_P2.54mm_Horizontal"
-			(at 68.58 69.85 0)
+			(at 68.58 67.31 0)
 			(effects
 				(font
@@
 		)
 		(property "Datasheet" "~"
-			(at 68.58 69.85 0)
+			(at 68.58 67.31 0)
 			(effects
 				(font
@@
 		)
 		(property "Description" "Generic connector, single row, 01x06, script generated"
-			(at 68.58 69.85 0)
+			(at 68.58 67.31 0)
 			(effects
 				(font

Commit message: update new
Connections:
- net +5V: now also ToF_Vorne_1.6 (Pin_6); no longer ToF_Vorne_1.1 (Pin_1)
- net GND: now also ToF_Vorne_1.5 (Pin_5); no longer ToF_Vorne_1.2 (Pin_2)
- net SCL: now also ToF_Vorne_1.4 (Pin_4); no longer ToF_Vorne_1.3 (Pin_3)
- net SDA: now also ToF_Vorne_1.3 (Pin_3); no longer ToF_Vorne_1.4 (Pin_4)
- net ToF_XS_0: now also ToF_Vorne_1.1 (Pin_1); no longer ToF_Vorne_1.6 (Pin_6)
Other:
- moved on the sheet: ToF_Vorne_1
Changed lines of the file:
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@@
 	(symbol
 		(lib_id "Connector:Conn_01x06_Socket")
-		(at 68.58 67.31 0)
-		(mirror y)
+		(at 68.58 69.85 180)
 		(unit 1)
 		(exclude_from_sim no)
@@
 		)
 		(property "Value" "Conn_01x06_Socket"
-			(at 69.215 77.47 0)
+			(at 69.215 59.69 0)
 			(effects
 				(font
@@
 		)
 		(property "Footprint" "Connector_PinSocket_2.54mm:PinSocket_1x06_P2.54mm_Horizontal"
-			(at 68.58 67.31 0)
+			(at 68.58 69.85 0)
 			(effects
 				(font
@@
 		)
 		(property "Datasheet" "~"
-			(at 68.58 67.31 0)
+			(at 68.58 69.85 0)
 			(effects
 				(font
@@
 		)
 		(property "Description" "Generic connector, single row, 01x06, script generated"
-			(at 68.58 67.31 0)
+			(at 68.58 69.85 0)
 			(effects
 				(font
