File: MainPlatine/MainPlatine.kicad_pcb (KiCad board)
At the start: 2 copper layers, 107.9 x 120 mm, 7 parts, among them U4 TB6612FNG, U5 TB6612FNG

Commit message: add new
Parts:
- added A1: Arduino_Nano_v2.x, Module:Arduino_Nano, F.Cu at (100.9, 149.9)
- added Bumper_1: Conn_01x02_Pin, JST:JST-XH-02-PACKAGE-LONG-PAD, F.Cu at (189.2, 48.2)
- added Bumper_2: Conn_01x02_Pin, JST:JST-XH-02-PACKAGE-LONG-PAD, F.Cu at (97.9, 48.3)
- added Colo_Alt1: Conn_01x05_Pin, JST:JST-XH-05-PACKAGE-LONG-PAD, B.Cu at (199.0, 69.2)
- added Color_NEU1: Conn_01x05_Pin, JST:JST-XH-05-PACKAGE-LONG-PAD, B.Cu at (191.0, 127.4)
- added Gyro1: Conn_01x05_Pin, JST:JST-XH-05-PACKAGE-LONG-PAD, B.Cu at (184.0, 127.4)
- added J1: Conn_01x07_Pin, JST:JST-XH-07-PACKAGE-LONG-PAD, F.Cu at (174.2, 150.6)
- added RB1: 10k, Resistor_SMD:R_1206_3216Metric_Pad1.30x1.75mm_HandSolder, B.Cu at (152.1, 65.8)
- added RB2: 10k, Resistor_SMD:R_1206_3216Metric_Pad1.30x1.75mm_HandSolder, B.Cu at (149.6, 65.8)
- added RI1: 10k, Resistor_SMD:R_1206_3216Metric_Pad1.30x1.75mm_HandSolder, F.Cu at (188.9, 117.1)
- added RI2: 10k, Resistor_SMD:R_1206_3216Metric_Pad1.30x1.75mm_HandSolder, F.Cu at (186.1, 117.1)
- added ToF_Vorne_1: Conn_01x06_Socket, Connector_PinSocket_2.54mm:PinSocket_1x06_P2.54mm_Horizontal, F.Cu at (149.6, 54.3)
- added U1: Main Conector to Main pcb, Robotik:Main Conetor, F.Cu at (144.6, 89.4)
- Motor1, Motor2: footprint Connector_PinSocket_2.54mm:PinSocket_1x06_P2.54mm_Vertical -> JST:JST-XH-06-PACKAGE-LONG-PAD; moved to B.Cu
- Motor3, Motor4: footprint Connector_PinSocket_2.54mm:PinSocket_1x06_P2.54mm_Vertical -> JST:JST-XH-06-PACKAGE-LONG-PAD
- moved U5 186.1 mm to (188.7, 140.8)
- moved Motor3 156.3 mm to (153.1, 150.7)
- moved U4 153.2 mm to (179.2, 49.9)
- moved Motor2 135.7 mm to (163.4, 48.1)
- moved Motor4 133.2 mm to (133.4, 150.6)
- moved Motor1 103.6 mm to (123.2, 48.1)
- moved B1 20.6 mm to (143.2, 82.9), turned to 0 degrees
Connections:
- B1 pad 14: unconnected-(B1-14(TX3)-Pad14) -> /ARD_RX_3
- B1 pad 15: unconnected-(B1-15(RX3)-Pad15) -> /ARD_TX_3
- B1 pad 16: unconnected-(B1-16(TX2)-Pad16) -> /ARD_TX_2
- B1 pad 17: unconnected-(B1-17(RX2)-Pad17) -> /ARD_RX_2
- B1 pad 18: unconnected-(B1-18(TX1)-Pad18) -> /ARD_TX_1
- B1 pad 19: unconnected-(B1-19(RX1)-Pad19) -> /ARD_RX_1
- B1 pad 2: unconnected-(B1-Pad2) -> /Bumper_Links
- B1 pad 20: unconnected-(B1-20(SDA)-Pad20) -> /SDA
- B1 pad 21: unconnected-(B1-21(SCL)-Pad21) -> /SCL
- B1 pad 23: /MOT_STBY -> /MOT2_IN1
- B1 pad 25: /MOT1_IN1 -> /MOT2_IN2
- B1 pad 27: /MOT1_IN2 -> /MOT_STBY
- B1 pad 29: /MOT2_IN1 -> /MOT1_IN2
- B1 pad 3: unconnected-(B1-Pad3) -> /Bumper_Rechts
- B1 pad 30: unconnected-(B1-Pad30) -> /Tof_XS_0
- B1 pad 31: /MOT2_IN2 -> /MOT1_IN1
- B1 pad 32: unconnected-(B1-Pad32) -> /Tof_XS_4
- B1 pad 33: /MOT3_IN1 -> /SW_SCL
- B1 pad 34: unconnected-(B1-Pad34) -> /Tof_XS_5
- B1 pad 35: /MOT3_IN2 -> /SW_SDA
- B1 pad 36: unconnected-(B1-Pad36) -> /Tof_XS_6
- B1 pad 37: /MOT4_IN1 -> /Tof_XS_1
- B1 pad 38: unconnected-(B1-Pad38) -> /LED_C2
- B1 pad 39: /MOT4_IN2 -> /Tof_XS_2
- B1 pad 40: unconnected-(B1-Pad40) -> /LED_C1
- B1 pad 41: unconnected-(B1-Pad41) -> /Tof_XS_3
- B1 pad 42: unconnected-(B1-Pad42) -> /UI_LED_2
- B1 pad 43: unconnected-(B1-Pad43) -> /MOT4_IN1
- B1 pad 44: unconnected-(B1-Pad44) -> /UI_LED_1
- B1 pad 45: unconnected-(B1-Pad45) -> /MOT4_IN2
- B1 pad 47: unconnected-(B1-Pad47) -> /MOT3_IN2
- B1 pad 49: unconnected-(B1-Pad49) -> /MOT3_IN1
- B1 pad 5V: unconnected-(B1-Pad5V) -> +5V
- B1 pad A0: unconnected-(B1-PadA0) -> /UI_Button_3
- B1 pad A1: unconnected-(B1-PadA1) -> /UI_Button_4
- B1 pad A10: unconnected-(B1-PadA10) -> /Encoder_B
- B1 pad A11: unconnected-(B1-PadA11) -> /Encoder_SW
- B1 pad A12: unconnected-(B1-PadA12) -> /Encoder_A
- B1 pad A13: unconnected-(B1-PadA13) -> /UI_Button_2
- B1 pad A14: unconnected-(B1-PadA14) -> /UI_Button_1
- B1 pad A15: unconnected-(B1-PadA15) -> /Color_Old_Interrupt
- B1 pad A8: unconnected-(B1-PadA8) -> /Interrupt_Cam1
- B1 pad A9: unconnected-(B1-PadA9) -> /Interrupt_Cam2
- B1 pad GND: unconnected-(B1-PadGND) -> GND
- Motor1 pad 1: /Treiber1/A+ -> /Treiber1/B+
- Motor1 pad 3: /ENC3_B -> /ENC2_B
- Motor1 pad 4: /ENC3_A -> /ENC2_A
- Motor1 pad 6: /Treiber1/A- -> /Treiber1/B-
- Motor2 pad 1: /Treiber1/B+ -> /Treiber1/A+
- Motor2 pad 3: /ENC4_B -> /ENC1_B
- Motor2 pad 4: /ENC4_A -> /ENC1_A
- Motor2 pad 6: /Treiber1/B- -> /Treiber1/A-
- Motor3 pad 1: /Treiber2/A+ -> /Treiber2/B+
- Motor3 pad 3: /ENC2_B -> /ENC4_B
- Motor3 pad 4: /ENC1_A -> /ENC4_A
- Motor3 pad 6: /Treiber2/A- -> /Treiber2/B-
- Motor4 pad 1: /Treiber2/B+ -> /Treiber2/A+
- Motor4 pad 3: /ENC2_B -> /ENC3_B
- Motor4 pad 4: /ENC2_A -> /ENC3_A
- Motor4 pad 6: /Treiber2/B- -> /Treiber2/A-
- U4 pad 11: /Treiber1/B+ -> /Treiber1/B-
- U4 pad 15: /MOT4_IN1 -> /MOT2_IN1
- U4 pad 16: /MOT4_PWM -> /MOT2_PWM
- U4 pad 17: /MOT4_IN2 -> /MOT2_IN2
- U4 pad 21: /MOT3_IN2 -> /MOT1_IN2
- U4 pad 22: /MOT3_PWM -> /MOT1_PWM
- U4 pad 23: /MOT3_IN1 -> /MOT1_IN1
- U4 pad 7: /Treiber1/B- -> /Treiber1/B+
- U5 pad 11: /Treiber2/B+ -> /Treiber2/B-
- U5 pad 15: /MOT2_IN1 -> /MOT4_IN1
- U5 pad 16: /MOT2_PWM -> /MOT4_PWM
- U5 pad 17: /MOT2_IN2 -> /MOT4_IN2
- U5 pad 21: /MOT1_IN2 -> /MOT3_IN2
- U5 pad 22: /MOT1_PWM -> /MOT3_PWM
- U5 pad 23: /MOT1_IN1 -> /MOT3_IN1
- U5 pad 7: /Treiber2/B- -> /Treiber2/B+
Routing:
- net +5V: track 0.00 -> 252.6 mm, vias 0 -> 1
- net GND: track 0.00 -> 214.1 mm, vias 0 -> 5
- net /SCL: track 0.00 -> 156.8 mm, vias 0 -> 1
- net /SDA: track 0.00 -> 143.7 mm, vias 0 -> 1
- net /ENC1_B: track 0.00 -> 138.8 mm
- net /ARD_TX_3: track 0.00 -> 136.1 mm
- net /ENC1_A: track 0.00 -> 134.6 mm
- net /ARD_RX_3: track 0.00 -> 131.0 mm
- net /MOT4_PWM: track 0.00 -> 113.5 mm, vias 0 -> 2
- net /MOT_STBY: track 0.00 -> 113.2 mm, vias 0 -> 1
- net /MOT3_PWM: track 0.00 -> 108.7 mm, vias 0 -> 2
- net /ENC2_B: track 0.00 -> 108.4 mm
- net /Tof_XS_1: track 0.00 -> 103.6 mm
- net /ENC2_A: track 0.00 -> 103.1 mm
- net /Tof_XS_3: track 0.00 -> 102.3 mm
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Other:
- board size 107.9 x 120 mm -> 121 x 111.5 mm
- copper layers 2 -> 4

Commit message: add main PCB
Parts:
- added J2: Conn_01x02_Pin, JST:JST-XH-02-PACKAGE-LONG-PAD, B.Cu at (192.7, 150.7)
- added J4: Conn_01x03_Pin, JST:JST-XH-03-PACKAGE-LONG-PAD, F.Cu at (89.5, 87.4)
- added PSU1: ~, Robotik:Untitled_1, F.Cu at (192.6, 133.2)
- moved Gyro1 68.6 mm to (116.9, 113.1), turned to 180 degrees
- moved J1 61.1 mm to (113.2, 150.6)
- moved RI1 53.9 mm to (177.3, 64.5), turned to 90 degrees
- moved RI2 52.9 mm to (180.2, 64.5), turned to 90 degrees
- moved Color_NEU1 26.5 mm to (168.4, 113.6), turned to 180 degrees
- moved U5 18.1 mm to (171.6, 146.7)
- moved U1 2.80 mm to (144.8, 86.6)
Connections:
- B1 pad 26: unconnected-(B1-Pad26) -> /LEDB_U
- B1 pad 28: unconnected-(B1-Pad28) -> /GYRO_RST
- B1 pad 50: unconnected-(B1-50/MISO-Pad50) -> /MISO
- B1 pad 51: unconnected-(B1-51/MOSI-Pad51) -> /MOSI
- B1 pad 52: unconnected-(B1-52/SCK-Pad52) -> /SCK
- Gyro1 pad 1: /Sensorik/Gyro_RST -> /GYRO_RST
- U1 pad D+: unconnected-(U1-Mega_D+-PadD+) -> /D+
- U1 pad D-: unconnected-(U1-Mega_D--PadD-) -> /D-
- U1 pad MOSI: unconnected-(U1-PadMOSI) -> /MISO
- U1 pad SCK: unconnected-(U1-PadSCK) -> /SCK
Routing:
- net GND: track 214.1 -> 655.8 mm, vias 5 -> 4
- net +5V: track 252.6 -> 535.7 mm, vias 1 -> 2
- net /6V: track 0.00 -> 161.5 mm, vias 0 -> 4
- net /GYRO_RST: track 0.00 -> 112.9 mm, vias 0 -> 2
- net /LEDB_U: track 0.00 -> 106.8 mm, vias 0 -> 1
- net /SCL: track 156.8 -> 252.5 mm, vias 1 -> 2
- net /SDA: track 143.7 -> 234.3 mm, vias 1 -> 0
- net /MOSI: track 0.00 -> 70.6 mm, vias 0 -> 1
- net /MISO: track 0.00 -> 62.4 mm, vias 0 -> 1
- net /SCK: track 0.00 -> 61.0 mm, vias 0 -> 2
- net /Tof_XS_2: track 97.2 -> 139.3 mm
- net /Tof_XS_1: track 103.6 -> 141.6 mm
- net /Tof_XS_3: track 102.3 -> 138.2 mm
- net /Treiber2/B+: track 58.4 -> 23.8 mm
- net /Treiber2/B-: track 28.5 -> 8.94 mm
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
Commit message: fix main pcb
Parts:
- added RI3: 10k, Resistor_SMD:R_1206_3216Metric_Pad1.30x1.75mm_HandSolder, B.Cu at (178.4, 80.4)
- added RI4: 10k, Resistor_SMD:R_1206_3216Metric_Pad1.30x1.75mm_HandSolder, B.Cu at (178.4, 83.4)
- moved Bumper_2 0.44 mm to (97.5, 48.2)
Connections:
- B1 pad 22: unconnected-(B1-Pad22) -> /LEDB_U
- B1 pad 24: unconnected-(B1-Pad24) -> /GYRO_RST
- B1 pad 26: /LEDB_U -> /IO_CAM2
- B1 pad 28: /GYRO_RST -> /IO_CAM1
- B1 pad 46: unconnected-(B1-Pad46) -> /D_D
- B1 pad 48: unconnected-(B1-Pad48) -> /Color_NEW_IO
- B1 pad 53: unconnected-(B1-53/~{CS}-Pad53) -> /CS_D
- B1 pad A7: unconnected-(B1-PadA7) -> /BAT_ADC
- ToF_Vorne_1 pad 1: /Tof_XS_0 -> +5V
- ToF_Vorne_1 pad 2: unconnected-(ToF_Vorne_1-Pin_2-Pad2) -> GND
- ToF_Vorne_1 pad 3: /SDA -> /SCL
- ToF_Vorne_1 pad 4: /SCL -> /SDA
- ToF_Vorne_1 pad 5: GND -> unconnected-(ToF_Vorne_1-Pin_5-Pad5)
- ToF_Vorne_1 pad 6: +5V -> /Tof_XS_0
- U1 pad CS_D: unconnected-(U1-CS_Display-PadCS_D) -> /CS_D
- U1 pad D_D: unconnected-(U1-D_Display-PadD_D) -> /D_D
- U1 pad R_C1: unconnected-(U1-Reset_Cam_1-PadR_C1) -> /IO_CAM1
- U1 pad R_C2: unconnected-(U1-Reset_Cam_2-PadR_C2) -> /IO_CAM2
Routing:
- net /CS_D: track 0.00 -> 81.3 mm, vias 0 -> 1
- net /D_D: track 0.00 -> 54.7 mm, vias 0 -> 1
- net /BAT_ADC: track 0.00 -> 46.9 mm, vias 0 -> 3
- net /Color_NEW_IO: track 0.00 -> 45.5 mm
- net /IO_CAM2: track 0.00 -> 44.6 mm
- net /IO_CAM1: track 0.00 -> 41.1 mm
- net GND: track 655.8 -> 691.8 mm
- net /Tof_XS_0: track 52.9 -> 68.0 mm
- net /6V: track 161.5 -> 166.8 mm
- net /MOSI: track 70.6 -> 75.2 mm
- net /LEDB_U: track 106.8 -> 110.3 mm
- net /MISO: track 62.4 -> 65.7 mm
- net /SCL: track 252.5 -> 249.6 mm
- net /SDA: track 234.3 -> 236.9 mm
- net /GYRO_RST: track 112.9 -> 115.0 mm
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
Commit message: update new
Parts:
- added RS_1: Conn_01x03_Pin, JST:JST-XH-03-PACKAGE-LONG-PAD, F.Cu at (88.5, 89.8)
- added RS_2: Conn_01x03_Pin, JST:JST-XH-03-PACKAGE-LONG-PAD, F.Cu at (88.5, 101.5)
- ToF_Vorne_1: moved to B.Cu
- moved ToF_Vorne_1 12.7 mm to (136.9, 54.1)
- moved J4 9.35 mm to (88.5, 78.1)
Connections:
- B1 pad 10: unconnected-(B1-Pad10) -> /RS_Servo_1
- B1 pad 8: unconnected-(B1-Pad8) -> /RES_D
- B1 pad 9: unconnected-(B1-Pad9) -> /RS_Servo_2
- ToF_Vorne_1 pad 1: +5V -> /Tof_XS_0
- ToF_Vorne_1 pad 2: GND -> unconnected-(ToF_Vorne_1-Pin_2-Pad2)
- ToF_Vorne_1 pad 3: /SCL -> /SDA
- ToF_Vorne_1 pad 4: /SDA -> /SCL
- ToF_Vorne_1 pad 5: unconnected-(ToF_Vorne_1-Pin_5-Pad5) -> GND
- ToF_Vorne_1 pad 6: /Tof_XS_0 -> +5V
- U1 pad 1: (no net) -> /RES_D
- U1 pad I_C1: /Interrupt_Cam2 -> unconnected-(U1-Interrupt_Cam_1-PadI_C1)
- U1 pad LED1: /LED_C2 -> unconnected-(U1-Beleuchtung_Cam_1-PadLED1)
- U1 pad RX_C1: /ARD_TX_1 -> unconnected-(U1-RX_Cam_1-PadRX_C1)
- U1 pad R_C1: /IO_CAM1 -> unconnected-(U1-Reset_Cam_1-PadR_C1)
- U1 pad TX_C1: /ARD_RX_1 -> unconnected-(U1-TX_Cam_1-PadTX_C1)
Routing:
- net /RS_Servo_2: track 0.00 -> 70.6 mm
- net /RS_Servo_1: track 0.00 -> 57.7 mm
- net +5V: track 536.3 -> 573.9 mm
- net /RES_D: track 0.00 -> 34.5 mm, vias 0 -> 1
- net GND: track 691.8 -> 696.8 mm
- net /LEDB_U: track 110.3 -> 107.5 mm

Commit message: read by lk
Routing:
- net GND: track 696.8 -> 708.9 mm
Changed lines of the file:
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@@
+	)
+	(segment
+		(start 88.5175 98.96)
+		(end 89.76 98.96)
+		(width 0.5)
+		(layer "B.Cu")
+		(net 1)
 	)
 	(segment
@@
 	)
 	(segment
+		(start 89.76 98.96)
+		(end 92.3 101.5)
+		(width 0.5)
+		(layer "B.Cu")
+		(net 1)
+	)
+	(segment
 		(start 129.5 154.5)
 		(end 149 154.5)
@@
 		(width 0.5)
 		(layer "B.Cu")
+		(net 1)
+	)
+	(segment
+		(start 94.98 107.68)
+		(end 92.3 105)
+		(width 0.5)
+		(layer "B.Cu")
+		(net 1)
+	)
+	(segment
+		(start 92.3 105)
+		(end 92.3 101.5)
+		(width 0.5)
+		(layer "B.Cu")
