File: UserInterface/button.kicad_sch (KiCad schematic)
At the start: 19 parts, among them SW0 RotaryEncoder_Switch_MP, SW1 SW_SPST, SW2 SW_SPST, SW3 SW_SPST, SW4 SW_SPST

Commit message: add new
Changed lines of the file:
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@@
-	(wire
-		(pts
-			(xy 127 113.03) (xy 125.73 113.03)
-		)
-		(stroke
-			(width 0)
-			(type default)
-		)
-	)
 	(wire
 		(pts
