File: UserInterface/UserInterface.kicad_sch (KiCad schematic)
At the start: 9 parts, among them J1 Conn_01x18_Pin

Commit message: add main PCB
Connections:
- net BUTTON_1: now also J1.13 (Pin_13); no longer J1.8 (Pin_8)
- net BUTTON_2: now also J1.14 (Pin_14); no longer J1.9 (Pin_9)
- net BUTTON_3: now also J1.15 (Pin_15); no longer J1.10 (Pin_10)
- net BUTTON_4: now also J1.16 (Pin_16); no longer J1.11 (Pin_11)
- net LED_A: now also J1.11 (Pin_11); no longer J1.15 (Pin_15)
- net LED_B: now also J1.12 (Pin_12); no longer J1.16 (Pin_16)
- net RE_A: now also J1.9 (Pin_9); no longer J1.13 (Pin_13)
- net RE_B: now also J1.10 (Pin_10); no longer J1.14 (Pin_14)
- net RE_SW: now also J1.8 (Pin_8); no longer J1.12 (Pin_12)
Changed lines of the file:
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@@
+		)
+	)
+	(label "RE_A"
+		(at 161.29 111.76 270)
+		(effects
+			(font
+				(size 1.27 1.27)
+			)
+			(justify right bottom)
+		)
+	)
+	(label "BUTTON_1"
+		(at 171.45 111.76 270)
+		(effects
+			(font
+				(size 1.27 1.27)
+			)
+			(justify right bottom)
 		)
 	)
@@
 		)
 	)
-	(label "BUTTON_4"
-		(at 166.37 111.76 270)
-		(effects
-			(font
-				(size 1.27 1.27)
-			)
-			(justify right bottom)
-		)
-	)
 	(label "LED_B"
 		(at 223.52 58.42 180)
@@
 		)
 	)
+	(label "RE_B"
+		(at 163.83 111.76 270)
+		(effects
+			(font
+				(size 1.27 1.27)
+			)
+			(justify right bottom)
+		)
+	)
 	(label "BUTTON_4"
 		(at 53.34 72.39 0)
@@
 		)
 	)
+	(label "BUTTON_2"
+		(at 173.99 111.76 270)
+		(effects
+			(font
+				(size 1.27 1.27)
+			)
+			(justify right bottom)
+		)
+	)
 	(label "RE_SW"
 		(at 101.6 63.5 180)
@@
 		)
 	)
-	(label "RE_A"
-		(at 171.45 111.76 270)
+	(label "BUTTON_4"
+		(at 179.07 111.76 270)
+		(effects
+			(font
+				(size 1.27 1.27)
+			)
+			(justify right bottom)
+		)
+	)
+	(label "LED_A"
+		(at 166.37 111.76 270)
 		(effects
 			(font
@@
 	)
 	(label "BUTTON_3"
-		(at 163.83 111.76 270)
-		(effects
-			(font
-				(size 1.27 1.27)
-			)
-			(justify right bottom)
-		)
-	)
-	(label "RE_B"
-		(at 173.99 111.76 270)
-		(effects
-			(font
-				(size 1.27 1.27)
-			)
-			(justify right bottom)
-		)
-	)
-	(label "LED_A"
 		(at 176.53 111.76 270)
 		(effects
@@
 		)
 	)
+	(label "LED_B"
+		(at 168.91 111.76 270)
+		(effects
+			(font
+				(size 1.27 1.27)
+			)
+			(justify right bottom)
+		)
+	)
 	(label "MOSI"
 		(at 55.88 106.68 0)
@@
 		)
 	)
-	(label "RE_SW"
-		(at 168.91 111.76 270)
-		(effects
-			(font
-				(size 1.27 1.27)
-			)
-			(justify right bottom)
-		)
-	)
-	(label "LED_B"
-		(at 179.07 111.76 270)
-		(effects
-			(font
-				(size 1.27 1.27)
-			)
-			(justify right bottom)
-		)
-	)
 	(label "D"
 		(at 55.88 102.87 0)
@@
 		)
 	)
-	(label "BUTTON_1"
-		(at 158.75 111.76 270)
-		(effects
-			(font
-				(size 1.27 1.27)
-			)
-			(justify right bottom)
-		)
-	)
 	(label "MOSI"
 		(at 146.05 111.76 270)
@@
 		)
 	)
-	(label "BUTTON_2"
-		(at 161.29 111.76 270)
-		(effects
-			(font
-				(size 1.27 1.27)
-			)
-			(justify right bottom)
-		)
-	)
 	(label "BUTTON_3"
 		(at 53.34 68.58 0)
@@
 		)
 	)
+	(label "RE_SW"
+		(at 158.75 111.76 270)
+		(effects
+			(font
+				(size 1.27 1.27)
+			)
+			(justify right bottom)
+		)
+	)

Commit message: ready to fix ui pcb
Parts:
- removed J1: Conn_01x18_Pin, Connector_PinHeader_2.54mm:PinHeader_1x18_P2.54mm_Vertical, symbol Connector:Conn_01x18_Pin
- added J2, J3: Conn_01x08_Pin, JST:JST-XH-08-PACKAGE-LONG-PAD, symbol Connector:Conn_01x08_Pin
Connections:
- net +5V: now also J2.8 (Pin_8)
- net BUTTON_1: now also J2.4 (Pin_4)
- net BUTTON_2: now also J2.5 (Pin_5)
- net BUTTON_3: now also J2.6 (Pin_6)
- net BUTTON_4: now also J2.7 (Pin_7)
- net GND: now also J2.1 (Pin_1)
- net LED_A: now also J2.2 (Pin_2)
- net LED_B: now also J2.3 (Pin_3)
- net MOSI: now also J3.1 (Pin_1)
- net RES: now also J3.4 (Pin_4)
- net RE_A: now also J3.6 (Pin_6)
- net RE_B: now also J3.8 (Pin_8)
- net RE_SW: now also J3.7 (Pin_7)
- net SCK: now also J3.2 (Pin_2)
- new net CS_D: J3.5 (Pin_5)
- new net D_D: J3.3 (Pin_3)
