File: Top_Platine/MainKamera.kicad_sch (KiCad schematic)
At the start: 6 parts, among them SW3 SW_SPST

Commit message: add main PCB
Parts:
- removed CAM_USB_IN1, CAM_USB_IN2, CAM_USB_OUT1, CAM_USB_OUT2: Conn_01x04_Pin, JST:JST-XH-04-PACKAGE-LONG-PAD, symbol Connector:Conn_01x04_Pin
- removed U1: ~, Robotik:Untitled, symbol RobotikV4:AZ8521-5
- added SWC2: SW_SPST, Connector_PinHeader_2.54mm:PinHeader_1x02_P2.54mm_Horizontal, symbol Switch:SW_SPST
- SWC1: renamed from SW3; footprint Connector_PinHeader_2.54mm:PinHeader_1x02_P2.54mm_Vertical -> Connector_PinHeader_2.54mm:PinHeader_1x02_P2.54mm_Horizontal
Connections:
- net VCC: now also SWC2.1 (A)
- net Kamera1/5V: now reaches SWC1.1 (A)
- new net Kamera2/5V: SWC2.2 (B)
- no-connect marks 0 -> 8
Other:
- sheet Kamera1 ports: added INT_{Camera}; removed Reset
- sheet Kamera2 ports: added INT_{Camera}; removed Reset
- moved on the sheet: SWC1
