File: Top_Platine/cam.kicad_sch (KiCad schematic)
At the start: 4 parts, among them SW1 SW_SPST

Commit message: add main PCB
Connections:
- net +3.3V: now also CAM1.17 (3.3V)
- net Interrupt: now also CAM1.30 (P10)
- net INT_{Camera}: now reaches CAM1.29 (P9)
- net Reset: no longer names the net of CAM1.32 (RST)
Changed lines of the file:
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@@
+	(wire
+		(pts
+			(xy 127 82.55) (xy 135.89 82.55)
+		)
+		(stroke
+			(width 0)
+			(type default)
+		)
+	)
 	(wire
 		(pts
@@
 	(wire
 		(pts
+			(xy 135.89 85.09) (xy 135.89 82.55)
+		)
+		(stroke
+			(width 0)
+			(type default)
+		)
+	)
+	(wire
+		(pts
 			(xy 218.44 81.28) (xy 218.44 93.98)
 		)
@@
 	(wire
 		(pts
-			(xy 133.35 93.98) (xy 137.16 93.98)
+			(xy 127 80.01) (xy 127 82.55)
 		)
 		(stroke
@@
 	(wire
 		(pts
+			(xy 137.16 85.09) (xy 135.89 85.09)
+		)
+		(stroke
+			(width 0)
+			(type default)
+		)
+	)
+	(wire
+		(pts
 			(xy 151.13 121.92) (xy 151.13 119.38)
 		)
@@
 		(pts
 			(xy 218.44 101.6) (xy 218.44 105.41)
+		)
+		(stroke
+			(width 0)
+			(type default)
+		)
+	)
+	(wire
+		(pts
+			(xy 167.64 102.87) (xy 170.18 102.87)
+		)
+		(stroke
+			(width 0)
+			(type default)
+		)
+	)
+	(wire
+		(pts
+			(xy 167.64 105.41) (xy 170.18 105.41)
 		)
 		(stroke
@@
 		)
 	)
+	(hierarchical_label "INT_{Camera}"
+		(shape input)
+		(at 170.18 102.87 0)
+		(effects
+			(font
+				(size 1.27 1.27)
+			)
+			(justify left)
+		)
+	)
 	(hierarchical_label "MISO"
 		(shape input)
@@
 	(hierarchical_label "Interrupt"
 		(shape bidirectional)
-		(at 180.34 69.85 0)
+		(at 170.18 105.41 0)
 		(effects
 			(font
@@
 		(shape input)
 		(at 218.44 115.57 270)
-		(effects
-			(font
-				(size 1.27 1.27)
-			)
-			(justify right)
-		)
-	)
-	(hierarchical_label "Reset"
-		(shape input)
-		(at 133.35 93.98 180)
 		(effects
 			(font
@@
 					(unit 1)
 				)
+			)
+		)
+	)
+	(symbol
+		(lib_id "power:+3.3V")
+		(at 127 80.01 0)
+		(unit 1)
+		(exclude_from_sim no)
+		(in_bom yes)
+		(on_board yes)
+		(dnp no)
+		(fields_autoplaced yes)
+		(property "Reference" "#PWR09"
+			(at 127 83.82 0)
+			(effects
+				(font
+					(size 1.27 1.27)
+				)
+				(hide yes)
+			)
+		)
+		(property "Value" "+3.3V"
+			(at 127 74.93 0)
+			(effects
+				(font
+					(size 1.27 1.27)
+				)
+			)
+		)
+		(property "Footprint" ""
+			(at 127 80.01 0)
+			(effects
+				(font
+					(size 1.27 1.27)
+				)
+				(hide yes)
+			)
+		)
+		(property "Datasheet" ""
+			(at 127 80.01 0)
+			(effects
+				(font
+					(size 1.27 1.27)
+				)
+				(hide yes)
+			)
+		)
+		(property "Description" "Power symbol creates a global label with name \"+3.3V\""
+			(at 127 80.01 0)
+			(effects
+				(font
+					(size 1.27 1.27)
+				)
+				(hide yes)
+			)
+		)
+		(pin "1"
+		)
+		(instances
+			(project "Top_Platine"
+				(path "/f9eddfb7-9f4e-4814-b89b-9cecdea203a8/4a0c0bf0-fc48-418f-bd7b-41269867e8f6/6c6966d1-cda9-459c-af60-53d343a22294"
+					(reference "#PWR010")
+					(unit 1)
+				)
+				(path "/f9eddfb7-9f4e-4814-b89b-9cecdea203a8/4a0c0bf0-fc48-418f-bd7b-41269867e8f6/7d003288-345a-4c04-ac5a-41602d9002f9"
+					(reference "#PWR09")
+					(unit 1)
+				)
