File: Top_Platine/Top_Platine.kicad_sch (KiCad schematic)
At the start: 2 parts, among them U2 Main Conector to Main pcb

Commit message: add main PCB
Parts:
- removed Userinterface1: Conn_01x18_Pin, Connector_PinHeader_2.54mm:PinHeader_1x18_P2.54mm_Vertical, symbol Connector:Conn_01x18_Pin
- added BLED1, BLED2: Conn_01x03_Pin, JST:JST-XH-03-PACKAGE-LONG-PAD, symbol Connector:Conn_01x03_Pin
- added J1, J2: Conn_01x08_Pin, JST:JST-XH-08-PACKAGE-LONG-PAD, symbol Connector:Conn_01x08_Pin
Connections:
- net +5V: now also BLED1.1 (Pin_1), BLED2.1 (Pin_1), J1.8 (Pin_8)
- net BUTTON_1: now also J1.4 (Pin_4)
- net BUTTON_2: now also J1.5 (Pin_5)
- net BUTTON_3: now also J1.6 (Pin_6)
- net BUTTON_4: now also J1.7 (Pin_7)
- net CS_C1: now also U2.CS_C1 (Chip_Select_Cam_1)
- net CS_C2: now also U2.CS_C2 (Chip_Select_Cam_2)
- net GND: now also BLED1.3 (Pin_3), BLED2.3 (Pin_3), J1.1 (Pin_1)
- net INT_C1: now also U2.I_C1 (Interrupt_Cam_1)
- net INT_C2: now also U2.I_C2 (Interrupt_Cam_2)
- net LED_A: now also J1.2 (Pin_2)
- net LED_B: now also J1.3 (Pin_3)
- net MOSI: now also U2.MOSI, J2.1 (Pin_1)
- net RES: now also J2.4 (Pin_4)
- net RE_A: now also J2.6 (Pin_6)
- net RE_B: now also J2.8 (Pin_8)
- net RE_SW: now also J2.7 (Pin_7)
- net RX_C1: now also U2.RX_C1 (RX_Cam_1)
- net RX_C2: now also U2.RX_C2 (RX_Cam_2)
- net SCK: now also U2.SCK, J2.2 (Pin_2)
- net TX_C1: now also U2.TX_C1 (TX_Cam_1)
- net TX_C2: now also U2.TX_C2 (TX_Cam_2)
- net CS_D: now reaches U2.CS_D (CS_Display)
- net CS_D: now also J2.5 (Pin_5)
- net D_D: now reaches U2.D_D (D_Display)
- net D_D: now also J2.3 (Pin_3)
- net BLED_C1: now reaches U2.LED1 (Beleuchtung_Cam_1)
- net BLED_C1: now also BLED1.2 (Pin_2)
- net BLED_C2: now reaches U2.LED2 (Beleuchtung_Cam_2)
- net BLED_C2: now also BLED2.2 (Pin_2)
- net MISO: now reaches U2.MISO
- net INTT_C1: now reaches U2.R_C1 (Reset_Cam_1)
- net INTT_C2: now reaches U2.R_C2 (Reset_Cam_2)
Other:
- sheet Kamera ports: added InterruptToCam1, InterruptToCam2; removed Reset1, Reset2
- note added: "RES!?"

Commit message: update new
Parts:
- added J3: Conn_01x04_Pin, JST:JST-XH-04-PACKAGE-LONG-PAD, symbol Connector:Conn_01x04_Pin
Connections:
- net +5V: now also J3.1 (Pin_1)
- net GND: now also J3.4 (Pin_4)
- net RES: now also U2.1 (RES_D)
- net at U2.D+ (Mega_D+): now also J3.2 (Pin_2)
- net at U2.D- (Mega_D-): now also J3.3 (Pin_3)
Other:
- note added: "LEVELSHIFTER!!!"
- note removed: "RES!?"

Commit message: ready to fix ui pcb
Other:
- note removed: "LEVELSHIFTER!!!"
Changed lines of the file:
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@@
 	(generator_version "9.0")
 	(paper "A4")
-	(text "LEVELSHIFTER!!!\n"
-		(exclude_from_sim no)
-		(at 164.084 156.464 0)
-		(effects
-			(font
-				(size 1.27 1.27)
-			)
-		)
-	)
 	(wire
 		(pts
